File: pcb_design/Frequency_Meter.kicad_sch (KiCad schematic)
At the start: 67 parts, among them IC1 LMH6624MA_NOPB, IC2 AD8611ARZ, IC3 74LVC1G74DC,125, IC6 STM32G431KBT6, IC7 REF3125AIDBZT, J2 USB4105-GF-A, J3 Conn_01x04_Pin, J4 RF2-03E-T-00-50-G, U1 USBLC6-2SC6, U2 AP2112K-3.3, Y1 ABM3B-16.000MHZ-10-1-U-T

Commit message: Update schematic
Parts:
- removed IC1: LMH6624MA_NOPB, FreqMeter:SOIC127P600X175-8N, symbol Frequency_Meter:LMH6624MA_NOPB
- added IC4: AD8021ARZ, SOIC127P600X175-8N, symbol Frequency_Meter:AD8021ARZ
Connections:
- net +IN: now also IC4.3 (+IN)
- net GND: now also IC4.1 (LOGIC_REFERENCE), IC4.4 (-VS)
- net LOOPBACK+: now also IC4.6 (VOUT)
- net LOOPBACK-: now also IC4.2 (-IN)
- net RF_5V: now also IC4.7 (+VS), IC4.8 (~{DISABLE})
- no-connect marks 22 -> 20
Other:
- note removed: "PI-type filter"
- moved on the sheet: C5

Commit message: Schematics update
Parts:
- removed C3: 33pF, Capacitor_SMD:C_0402_1005Metric, symbol Device:C
- removed IC2: AD8611ARZ, FreqMeter:SOIC127P600X175-8N, symbol Frequency_Meter:AD8611ARZ
- removed IC3: 74LVC1G74DC,125, FreqMeter:SOP50P310X100-8N, symbol Frequency_Meter:74LVC1G74DC,125
- removed IC4: AD8021ARZ, SOIC127P600X175-8N, symbol Frequency_Meter:AD8021ARZ
- removed IC7: REF3125AIDBZT, FreqMeter:SOT95P237X112-3N, symbol Frequency_Meter:REF3125AIDBZT
- removed J4: RF2-03E-T-00-50-G, FreqMeter:RF203ET0050G, symbol Frequency_Meter:RF2-03E-T-00-50-G
- removed R14: 330k, Resistor_SMD:R_0603_1608Metric, symbol Device:R
- added C11, C28: 18pF, Capacitor_SMD:C_0603_1608Metric, symbol Device:C
- added C12, C29, C30: 15pF, Capacitor_SMD:C_0603_1608Metric, symbol Device:C
- added C27: 1uF X7R, Capacitor_SMD:C_0805_2012Metric, symbol Device:C
- added DS1: OLED_128X64_1.3_I2C, Screens:LCD_OLED_128X64_1.3_I2C, symbol Screens:OLED_128X64_1.3_I2C
- added IC1: LMH6629MF_NOPB, FreqMeter:SOT95P280X145-5N, symbol Frequency_Meter:LMH6629MF_NOPB
- added IC2: SN74LVC1G80DBVR, FreqMeter:SOT95P280X145-5N, symbol Frequency_Meter:SN74LVC1G80DBVR
- added IC3: REF2033AIDDCT, FreqMeter:SOT95P280X110-5N, symbol Frequency_Meter:REF2033AIDDCT
- added IC4: TLV3601DBVR, FreqMeter:SOT95P280X145-5N, symbol Frequency_Meter:TLV3601DBVR
- added J1: SMA female 50Ω edge mount, Connector_Coaxial:SMA_Amphenol_132289_EdgeMount, symbol Connector:Conn_Coaxial
- C1: value 33pF -> 15pF; footprint Capacitor_SMD:C_0402_1005Metric -> Capacitor_SMD:C_0603_1608Metric
- C2: value 130pF -> 100pF; footprint Capacitor_SMD:C_0402_1005Metric -> Capacitor_SMD:C_0603_1608Metric
- C22, C23: footprint Capacitor_SMD:C_0402_1005Metric -> Capacitor_SMD:C_0603_1608Metric
- DNP_R1, DNP_R2, R1: footprint Capacitor_SMD:C_0603_1608Metric -> Resistor_SMD:R_0603_1608Metric
- R10: value 33 Ohm -> 33
- R4: value 10k -> 1k
- R5: value 249 -> 374
Connections:
- net CLK_100M: now also IC2.2 (CLK)
- net CLK_DIV2: now also IC2.1 (D), IC2.4 (~{Q})
- net FILTER_OUT: now also C12.2, C28.2
- net GND: now also C9.2, C27.1, C29.1, C30.1, IC1.2 (V-), IC2.3 (GND), IC3.2 (GND), IC4.2 (VEE), J1.2 (Ext); no longer C9.1
- net POWER_3V3: now also C9.1, FB1.1, IC2.5 (VCC), IC4.5 (VCC)
- net POWER_5V: now also C26.1, C27.2, IC3.3 (EN), IC3.4 (VIN); no longer FB1.1
- net RF_IN: now also J1.1 (In)
- net at C1.1, L1.2: now also C11.1
- net at C1.2, C2.1, L3.1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: now also C11.2, C29.2, C30.2
- net at R10.1: now also IC4.1 (OUT)
- net at L3.2: now also C12.1, C28.1
- net +IN renamed AMP_+IN
- net AMP_+IN: now also IC1.3 (+IN)
- net -_NODE renamed COMPARATOR_IN-
- net COMPARATOR_IN-: now also IC4.4 (IN-)
- net COMPARATOR_IN+: no longer names the net of R8.2
- net COMPARATOR_IN+: now also IC4.3 (IN+)
- net LOOPBACK+ renamed AMP_OUT
- net AMP_OUT: now also IC1.1 (OUT)
- net LOOPBACK- renamed AMP_-IN
- net AMP_-IN: now also IC1.4 (-IN)
- net RF_5V renamed RF_3V3
- net RF_3V3: now also IC1.5 (V+); no longer C26.1, C9.2
- net VREF_2V5 renamed VREF_1V6
- net VREF_1V6: now also IC3.1 (VBIAS)
- no-connect marks 20 -> 19
Other:
- note added: "Built-in hysteresis 3mV"
- note removed: "f0 = sqrt(50*100) ~ 70,7 MHz f0 = 1/(2*PI*sqrt(LC))"
- moved on the sheet: C1, C10, C2, C25, C4, C5, C6, C7, C8, C9, L1, L3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
